File: pcb/eagleCad/goJAMMAv02.brd (EAGLE design)
At the start: 110 x 72 mm, 111 parts, among them IC1 MCP3004-I_SL, IC2 THS7314D, J1 DM3AT-SF-PEJM5, U1 +3.3v REG, U10 SN74HC245PWR, U11 SN74HC245PWR, U12 SN74HC245PWR, U13 IS61WV10248EDBLL-10TLI, U14 IS66WVH16M8BLL-100B1LI, U4 PCM5101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

Commit message: Add files via upload
Parts:
- C1, C2: value 10nF -> 100nF
- C12, C13, C17, C21: value 1mF -> 100uF
- C16, C4, C5, C7: value 100n -> 100nF
- R12, R13, R5: value 75R -> 0R
- R2: value 1K -> 150R
- R8: value 1K -> 560R
- U2: value (none) -> +1.8v REG
Other:
- board text removed: "BONEYARD"
- board text removed: "expansion"
