File: pcb/eagleCad/goJAMMAv02.sch (EAGLE design)
At the start: 107 parts, among them IC1 MCP3004-I_SL, IC2 THS7314D, J1 DM3AT-SF-PEJM5, U1 +3.3v REG, U10 SN74HC245PWR, U11 SN74HC245PWR, U12 SN74HC245PWR, U13 IS61WV10248EDBLL-10TLI, U14 IS66WVH16M8BLL-100B1LI, U4 PCM5101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

Commit message: Add files via upload
Parts:
- C1, C2: value 10nF -> 100nF
- C12, C13, C17, C21: value 1mF -> 100uF
- C16, C4, C5, C7: value 100n -> 100nF
- R12, R13, R5: value 75R -> 0R
- R2: value 1K -> 150R
- R8: value 1K -> 560R
- U2: value (none) -> +1.8v REG
Changed lines of the file:
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@@
 <?xml version="1.0" encoding="utf-8"?>
 <!DOCTYPE eagle SYSTEM "eagle.dtd">
-<eagle version="9.2.2">
+<eagle version="9.3.1">
 <drawing>
 <settings>
@@
 <part name="BUT5_6" library="con-lstb" library_urn="urn:adsk.eagle:library:162" deviceset="MA03-2" device="" package3d_urn="urn:adsk.eagle:package:8334/1"/>
 <part name="GND17" library="supply1" library_urn="urn:adsk.eagle:library:371" deviceset="GND" device=""/>
-<part name="C21" library="SparkFun-Capacitors" library_urn="urn:adsk.eagle:library:510" deviceset="1000UF" device="-RADIAL-5MM-25V-20%" package3d_urn="urn:adsk.eagle:package:37412/1" value="1mF"/>
+<part name="C21" library="SparkFun-Capacitors" library_urn="urn:adsk.eagle:library:510" deviceset="1000UF" device="-RADIAL-5MM-25V-20%" package3d_urn="urn:adsk.eagle:package:37412/1" value="100uF"/>
 <part name="U4" library="cronic" deviceset="PCM5101" device=""/>
 <part name="C9" library="rcl" deviceset="C-EU" device="C0805K" value="2u2"/>
 <part name="C10" library="rcl" deviceset="C-EU" device="C0805K" value="2u2"/>
-<part name="C4" library="rcl" deviceset="C-EU" device="C0805K" value="100n"/>
+<part name="C4" library="rcl" deviceset="C-EU" device="C0805K" value="100nF"/>
 <part name="GND18" library="supply1" deviceset="GND" device=""/>
 <part name="GND19" library="supply1" deviceset="GND" device=""/>
 <part name="R9" library="rcl" deviceset="R-EU_" device="R0805" value="1K"/>
 <part name="R11" library="rcl" deviceset="R-EU_" device="R0805" value="1K"/>
-<part name="C5" library="rcl" deviceset="C-EU" device="C0805K" value="100n"/>
+<part name="C5" library="rcl" deviceset="C-EU" device="C0805K" value="100nF"/>
 <part name="GND20" library="supply1" deviceset="GND" device=""/>
 <part name="R3" library="rcl" deviceset="R-EU_" device="R0805" value="1K"/>
 <part name="R4" library="rcl" deviceset="R-EU_" device="R0805" value="1K"/>
 <part name="GND21" library="supply1" deviceset="GND" device=""/>
-<part name="C7" library="rcl" deviceset="C-EU" device="C0805K" value="100n"/>
+<part name="C7" library="rcl" deviceset="C-EU" device="C0805K" value="100nF"/>
 <part name="C28" library="rcl" deviceset="C-EU" device="C0805K" value="100n"/>
 <part name="U3" library="jammaFPGA" deviceset="LM4755" device=""/>
-<part name="C1" library="rcl" deviceset="C-EU" device="C0805K" value="10nF"/>
-<part name="C2" library="rcl" deviceset="C-EU" device="C0805K" value="10nF"/>
+<part name="C1" library="rcl" deviceset="C-EU" device="C0805K" value="100nF"/>
+<part name="C2" library="rcl" deviceset="C-EU" device="C0805K" value="100nF"/>
 <part name="C3" library="SparkFun-Capacitors" library_urn="urn:adsk.eagle:library:510" deviceset="100UF-POLAR" device="-RADIAL-2.5MM-25V-20%" package3d_urn="urn:adsk.eagle:package:37415/1" value="100uF"/>
 <part name="GND22" library="supply1" library_urn="urn:adsk.eagle:library:371" deviceset="GND" device=""/>
@@
 <part name="GND28" library="supply1" library_urn="urn:adsk.eagle:library:371" deviceset="GND" device=""/>
 <part name="U1" library="SparkFun-IC-Power" deviceset="V_REG_78XX" device="7812" value="+3.3v REG"/>
-<part name="C12" library="SparkFun-Capacitors" library_urn="urn:adsk.eagle:library:510" deviceset="1000UF" device="-RADIAL-5MM-25V-20%" package3d_urn="urn:adsk.eagle:package:37412/1" value="1mF"/>
-<part name="C13" library="SparkFun-Capacitors" library_urn="urn:adsk.eagle:library:510" deviceset="1000UF" device="-RADIAL-5MM-25V-20%" package3d_urn="urn:adsk.eagle:package:37412/1" value="1mF"/>
-<part name="C16" library="rcl" deviceset="C-EU" device="C0805K" value="100n"/>
-<part name="U2" library="SparkFun-IC-Power" deviceset="V_REG_LM1117" device="SOT223"/>
-<part name="C17" library="SparkFun-Capacitors" library_urn="urn:adsk.eagle:library:510" deviceset="1000UF" device="-RADIAL-5MM-25V-20%" package3d_urn="urn:adsk.eagle:package:37412/1" value="1mF"/>
+<part name="C12" library="SparkFun-Capacitors" library_urn="urn:adsk.eagle:library:510" deviceset="1000UF" device="-RADIAL-5MM-25V-20%" package3d_urn="urn:adsk.eagle:package:37412/1" value="100uF"/>
+<part name="C13" library="SparkFun-Capacitors" library_urn="urn:adsk.eagle:library:510" deviceset="1000UF" device="-RADIAL-5MM-25V-20%" package3d_urn="urn:adsk.eagle:package:37412/1" value="100uF"/>
+<part name="C16" library="rcl" deviceset="C-EU" device="C0805K" value="100nF"/>
+<part name="U2" library="SparkFun-IC-Power" deviceset="V_REG_LM1117" device="SOT223" value="+1.8v REG"/>
+<part name="C17" library="SparkFun-Capacitors" library_urn="urn:adsk.eagle:library:510" deviceset="1000UF" device="-RADIAL-5MM-25V-20%" package3d_urn="urn:adsk.eagle:package:37412/1" value="100uF"/>
 <part name="LED1" library="led" library_urn="urn:adsk.eagle:library:259" deviceset="LED" device="CHIPLED_0805" package3d_urn="urn:adsk.eagle:package:15821/2"/>
 <part name="R1" library="rcl" deviceset="R-EU_" device="R0805" value="1K"/>
 <part name="LED2" library="led" library_urn="urn:adsk.eagle:library:259" deviceset="LED" device="CHIPLED_0805" package3d_urn="urn:adsk.eagle:package:15821/2"/>
 <part name="LED3" library="led" library_urn="urn:adsk.eagle:library:259" deviceset="LED" device="CHIPLED_0805" package3d_urn="urn:adsk.eagle:package:15821/2"/>
-<part name="R2" library="rcl" deviceset="R-EU_" device="R0805" value="1K"/>
-<part name="R8" library="rcl" deviceset="R-EU_" device="R0805" value="1K"/>
+<part name="R2" library="rcl" deviceset="R-EU_" device="R0805" value="150R"/>
+<part name="R8" library="rcl" deviceset="R-EU_" device="R0805" value="560R"/>
 <part name="GND30" library="supply1" library_urn="urn:adsk.eagle:library:371" deviceset="GND" device=""/>
 <part name="UART3_3V" library="con-lstb" library_urn="urn:adsk.eagle:library:162" deviceset="MA03-1" device="" package3d_urn="urn:adsk.eagle:package:8339/1"/>
@@
 <part name="IC2" library="SamacSys_Parts" deviceset="THS7314D" device=""/>
 <part name="GND32" library="supply1" library_urn="urn:adsk.eagle:library:371" deviceset="GND" device=""/>
-<part name="R5" library="rcl" deviceset="R-EU_" device="R0805" value="75R"/>
-<part name="R12" library="rcl" deviceset="R-EU_" device="R0805" value="75R"/>
-<part name="R13" library="rcl" deviceset="R-EU_" device="R0805" value="75R"/>
+<part name="R5" library="rcl" deviceset="R-EU_" device="R0805" value="0R"/>
+<part name="R12" library="rcl" deviceset="R-EU_" device="R0805" value="0R"/>
+<part name="R13" library="rcl" deviceset="R-EU_" device="R0805" value="0R"/>
 <part name="R14" library="rcl" deviceset="R-EU_" device="R0805" value="3K3"/>
 <part name="R15" library="rcl" deviceset="R-EU_" device="R0805" value="3K3"/>
@@
 <instance part="C1" gate="G$1" x="335.28" y="104.14" smashed="yes" rot="R90">
 <attribute name="NAME" x="335.28" y="109.22" size="1.778" layer="95" rot="R180"/>
-<attribute name="VALUE" x="342.9" y="96.52" size="1.778" layer="96" rot="R180"/>
+<attribute name="VALUE" x="345.44" y="109.22" size="1.778" layer="96" rot="R180"/>
 </instance>
 <instance part="C2" gate="G$1" x="335.28" y="99.06" smashed="yes" rot="R90">
 <attribute name="NAME" x="335.28" y="96.52" size="1.778" layer="95" rot="R180"/>
-<attribute name="VALUE" x="342.9" y="109.22" size="1.778" layer="96" rot="R180"/>
+<attribute name="VALUE" x="345.44" y="96.52" size="1.778" layer="96" rot="R180"/>
 </instance>
 <instance part="C3" gate="G$1" x="345.44" y="91.44" smashed="yes" rot="R270">
@@
 <instance part="U2" gate="G$1" x="134.62" y="86.36" smashed="yes">
 <attribute name="NAME" x="132.08" y="91.44" size="1.778" layer="95" rot="R180"/>
-<attribute name="VALUE" x="137.16" y="76.2" size="1.778" layer="96"/>
+<attribute name="VALUE" x="147.32" y="91.44" size="1.778" layer="96" rot="R180"/>
 </instance>
 <instance part="C17" gate="G$1" x="22.86" y="78.74" smashed="yes">
